File: Printed-Circuit-Boards/Prototyping-PCBs/Breadboard-Single/Breadboard.sch (EAGLE design)
At the start: 98 parts

Commit message: Updated PCB files.
Parts:
- added J45, J46, J47, J48, J49, J50: (no value), SparkFun-Connectors:CONN_05
- added J51, J52, J53, J54: 455-1750-1-ND, SparkFun-Connectors:CONN_03
Connections:
- new net N$75: J48.1, J48.2, J48.3, J48.4, J48.5
- new net N$76: J45.1, J45.2, J45.3, J45.4, J45.5
- new net N$77: J46.1, J46.2, J46.3, J46.4, J46.5
- new net N$78: J47.1, J47.2, J47.3, J47.4, J47.5
- new net N$79: J49.1, J49.2, J49.3, J49.4, J49.5
- new net N$80: J50.1, J50.2, J50.3, J50.4, J50.5
- net N$1: now also J52.1, J52.2, J52.3
- net N$2: now also J51.1, J51.2, J51.3
- net N$3: now also J54.1, J54.2, J54.3
- net N$4: now also J53.1, J53.2, J53.3
Other:
- moved on the sheet: J1, J10, J100, J101, J102, J103, J104, J105, J106, J107, J108, J109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
